Commit message: fixed odometry ros topic

File: app/robots/CER01/cer.urdf (robot description, URDF)
Before this commit: robot SIM_CER_ROBOT, 49 links, 48 joints
Joints:
- joint lidar_fixed_joint: origin xyz=0.0 0 0.0 rpy=0 0 0 -> xyz=0.0 0 1.0 rpy=0 0 0; parent base_link -> mobile_base_body

Commit message: Configuration update

File: app/robots/CER01/cer.urdf (robot description, URDF)
Before this commit: robot SIM_CER_ROBOT, 49 links, 48 joints
Joints:
- joint lidar_fixed_joint: origin xyz=0.0 0 1.0 rpy=0 0 0 -> xyz=0.3 0 0.1  rpy=0 0 0
