Commit message: urdf update

File: app/robots/CER01/cer.urdf (robot description, URDF)
Before this commit: robot SIM_CER_ROBOT, 49 links, 48 joints
Links:
- removed link base_center
- removed link head
- removed link l_clavicle
- removed link l_forearm
- removed link l_hand_paddle
- removed link l_hand_root
- removed link l_hand_thumb
- removed link l_shoulder
- removed link l_upperarm
- removed link l_wrist_tripod_base
- removed link l_wrist_tripod_pin_eq
- removed link l_wrist_tripod_slider_eq
- removed link left_camera
- removed link lidar
- removed link mobile_base_body
- removed link mobile_base_l_tyre
- removed link mobile_base_r_tyre
- removed link neck
- removed link oriented_xbk_yrg_zup_torso_tripod_platform
- removed link oriented_xfw_ylf_zup_torso_tripod_platform
- removed link r_clavicle
- removed link r_forearm
- removed link r_hand_paddle
- removed link r_hand_root
- removed link r_hand_thumb
- removed link r_shoulder
- removed link r_upperarm
- removed link r_wrist_tripod_base
- removed link r_wrist_tripod_pin_eq
- removed link r_wrist_tripod_slider_eq
- removed link right_camera
- removed link torso_chest
- removed link torso_tripod_pin_eq
- removed link torso_tripod_platform
- removed link torso_tripod_slider_eq
- added link base_laser
- added link chest_link, mass 13.0; collision mesh filename=package://cer_rviz/../../../cer-gazebo/cer2/meshes/dae/sim_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 scale=0.001 0.001 0.001; visual mesh filename=package://cer_rviz/../../../cer-gazebo/cer2/meshes/dae/sim_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 scale=0.001 0.001 0.001
- added link head_link, mass 2.0; collision mesh filename=package://cer_rviz/../../../cer-gazebo/cer2/meshes/dae/sim_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 scale=0.001 0.001 0.001; visual mesh filename=package://cer_rviz/../../../cer-gazebo/cer2/meshes/dae/sim_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 scale=0.001 0.001 0.001
- added link l_clavicle_link, mass 0.2; collision mesh filename=package://cer_rviz/../../../cer-gazebo/cer2/meshes/dae/sim_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 scale=0.001 0.001 0.001; visual mesh filename=package://cer_rviz/../../../cer-gazebo/cer2/meshes/dae/sim_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 scale=0.001 0.001 0.001
- added link l_elbow_sphere_link, mass 0.2; collision mesh filename=package://cer_rviz/../../../cer-gazebo/cer2/meshes/dae/sim_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 scale=0.001 0.001 0.001; visual mesh filename=package://cer_rviz/../../../cer-gazebo/cer2/meshes/dae/sim_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 scale=0.001 0.001 0.001
- added link l_forearm_link, mass 0.6; collision mesh filename=package://cer_rviz/../../../cer-gazebo/cer2/meshes/dae/sim_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 scale=0.001 0.001 0.001; visual mesh filename=package://cer_rviz/../../../cer-gazebo/cer2/meshes/dae/sim_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 scale=0.001 0.001 0.001
- added link l_hand_paddle_distal_link, mass 0.05; collision mesh filename=package://cer_rviz/../../../cer-gazebo/cer2/meshes/dae/sim_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 scale=0.001 0.001 0.001; visual mesh filename=package://cer_rviz/../../../cer-gazebo/cer2/meshes/dae/sim_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 scale=0.001 0.001 0.001
- added link l_hand_paddle_proximal_link, mass 0.05; collision mesh filename=package://cer_rviz/../../../cer-gazebo/cer2/meshes/dae/sim_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 scale=0.001 0.001 0.001; visual mesh filename=package://cer_rviz/../../../cer-gazebo/cer2/meshes/dae/sim_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 scale=0.001 0.001 0.001
- added link l_hand_root_link, mass 0.3; collision mesh filename=package://cer_rviz/../../../cer-gazebo/cer2/meshes/dae/sim_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 scale=0.001 0.001 0.001; visual mesh filename=package://cer_rviz/../../../cer-gazebo/cer2/meshes/dae/sim_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 scale=0.001 0.001 0.001
- added link l_hand_thumb_distal_link, mass 0.05; collision mesh filename=package://cer_rviz/../../../cer-gazebo/cer2/meshes/dae/sim_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 scale=0.001 0.001 0.001; visual mesh filename=package://cer_rviz/../../../cer-gazebo/cer2/meshes/dae/sim_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 scale=0.001 0.001 0.001
- added link l_hand_thumb_proximal_link, mass 0.05; collision mesh filename=package://cer_rviz/../../../cer-gazebo/cer2/meshes/dae/sim_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 scale=0.001 0.001 0.001; visual mesh filename=package://cer_rviz/../../../cer-gazebo/cer2/meshes/dae/sim_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 scale=0.001 0.001 0.001
- added link l_shoulder_link, mass 0.5; collision mesh filename=package://cer_rviz/../../../cer-gazebo/cer2/meshes/dae/sim_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 scale=0.001 0.001 0.001; visual mesh filename=package://cer_rviz/../../../cer-gazebo/cer2/meshes/dae/sim_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 scale=0.001 0.001 0.001
- added link l_upperarm_FT_sensor_frame
- added link l_upperarm_FT_sensor_link, mass 0.3; collision mesh filename=package://cer_rviz/../../../cer-gazebo/cer2/meshes/dae/sim_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 scale=0.001 0.001 0.001; visual mesh filename=package://cer_rviz/../../../cer-gazebo/cer2/meshes/dae/sim_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 scale=0.001 0.001 0.001
- added link l_upperarm_link, mass 0.5; collision mesh filename=package://cer_rviz/../../../cer-gazebo/cer2/meshes/dae/sim_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 scale=0.001 0.001 0.001; visual mesh filename=package://cer_rviz/../../../cer-gazebo/cer2/meshes/dae/sim_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 scale=0.001 0.001 0.001
- added link l_wrist_cup_eq_link, mass 0.2; collision mesh filename=package://cer_rviz/../../../cer-gazebo/cer2/meshes/dae/sim_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 scale=0.001 0.001 0.001; visual mesh filename=package://cer_rviz/../../../cer-gazebo/cer2/meshes/dae/sim_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 scale=0.001 0.001 0.001
- added link l_wrist_slider_eq_link, mass 0.3; collision mesh filename=package://cer_rviz/../../../cer-gazebo/cer2/meshes/dae/sim_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 scale=0.001 0.001 0.001; visual mesh filename=package://cer_rviz/../../../cer-gazebo/cer2/meshes/dae/sim_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 scale=0.001 0.001 0.001
- added link mobile_base_body_link, mass 14.0; collision mesh filename=package://cer_rviz/../../../cer-gazebo/cer2/meshes/dae/sim_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 scale=0.001 0.001 0.001; visual mesh filename=package://cer_rviz/../../../cer-gazebo/cer2/meshes/dae/sim_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 scale=0.001 0.001 0.001
- added link mobile_base_l_tyre_link, mass 3.0; collision cylinder length=0.06 radius=0.16; visual mesh filename=package://cer_rviz/../../../cer-gazebo/cer2/meshes/dae/sim_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 scale=0.001 0.001 0.001
- added link mobile_base_r_tyre_link, mass 3.0; collision cylinder length=0.06 radius=0.16; visual mesh filename=package://cer_rviz/../../../cer-gazebo/cer2/meshes/dae/sim_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 scale=0.001 0.001 0.001
- added link multicamera_sensor
- added link neck_link, mass 1.4; collision mesh filename=package://cer_rviz/../../../cer-gazebo/cer2/meshes/dae/sim_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 scale=0.001 0.001 0.001; visual mesh filename=package://cer_rviz/../../../cer-gazebo/cer2/meshes/dae/sim_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 scale=0.001 0.001 0.001
- added link oriented_xbk_yrg_zup_torso_platform
- added link oriented_xfw_ylf_zup_torso_platform
- added link r_clavicle_link, mass 0.2; collision mesh filename=package://cer_rviz/../../../cer-gazebo/cer2/meshes/dae/sim_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 scale=0.001 0.001 0.001; visual mesh filename=package://cer_rviz/../../../cer-gazebo/cer2/meshes/dae/sim_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 scale=0.001 0.001 0.001
- added link r_elbow_sphere_link, mass 0.2; collision mesh filename=package://cer_rviz/../../../cer-gazebo/cer2/meshes/dae/sim_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 scale=0.001 0.001 0.001; visual mesh filename=package://cer_rviz/../../../cer-gazebo/cer2/meshes/dae/sim_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 scale=0.001 0.001 0.001
- added link r_forearm_link, mass 0.6; collision mesh filename=package://cer_rviz/../../../cer-gazebo/cer2/meshes/dae/sim_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 scale=0.001 0.001 0.001; visual mesh filename=package://cer_rviz/../../../cer-gazebo/cer2/meshes/dae/sim_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 scale=0.001 0.001 0.001
- added link r_hand_paddle_distal_link, mass 0.05; collision mesh filename=package://cer_rviz/../../../cer-gazebo/cer2/meshes/dae/sim_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 scale=0.001 0.001 0.001; visual mesh filename=package://cer_rviz/../../../cer-gazebo/cer2/meshes/dae/sim_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 scale=0.001 0.001 0.001
- added link r_hand_paddle_proximal_link, mass 0.05; collision mesh filename=package://cer_rviz/../../../cer-gazebo/cer2/meshes/dae/sim_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 scale=0.001 0.001 0.001; visual mesh filename=package://cer_rviz/../../../cer-gazebo/cer2/meshes/dae/sim_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 scale=0.001 0.001 0.001
- added link r_hand_root_link, mass 0.3; collision mesh filename=package://cer_rviz/../../../cer-gazebo/cer2/meshes/dae/sim_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 scale=0.001 0.001 0.001; visual mesh filename=package://cer_rviz/../../../cer-gazebo/cer2/meshes/dae/sim_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 scale=0.001 0.001 0.001
- added link r_hand_thumb_distal_link, mass 0.05; collision mesh filename=package://cer_rviz/../../../cer-gazebo/cer2/meshes/dae/sim_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 scale=0.001 0.001 0.001; visual mesh filename=package://cer_rviz/../../../cer-gazebo/cer2/meshes/dae/sim_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 scale=0.001 0.001 0.001
- added link r_hand_thumb_proximal_link, mass 0.05; collision mesh filename=package://cer_rviz/../../../cer-gazebo/cer2/meshes/dae/sim_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 scale=0.001 0.001 0.001; visual mesh filename=package://cer_rviz/../../../cer-gazebo/cer2/meshes/dae/sim_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 scale=0.001 0.001 0.001
- added link r_shoulder_link, mass 0.5; collision mesh filename=package://cer_rviz/../../../cer-gazebo/cer2/meshes/dae/sim_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 scale=0.001 0.001 0.001; visual mesh filename=package://cer_rviz/../../../cer-gazebo/cer2/meshes/dae/sim_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 scale=0.001 0.001 0.001
- added link r_upperarm_FT_sensor_frame
- added link r_upperarm_FT_sensor_link, mass 0.3; collision mesh filename=package://cer_rviz/../../../cer-gazebo/cer2/meshes/dae/sim_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 scale=0.001 0.001 0.001; visual mesh filename=package://cer_rviz/../../../cer-gazebo/cer2/meshes/dae/sim_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 scale=0.001 0.001 0.001
- added link r_upperarm_link, mass 0.5; collision mesh filename=package://cer_rviz/../../../cer-gazebo/cer2/meshes/dae/sim_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 scale=0.001 0.001 0.001; visual mesh filename=package://cer_rviz/../../../cer-gazebo/cer2/meshes/dae/sim_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 scale=0.001 0.001 0.001
- added link r_wrist_cup_eq_link, mass 0.2; collision mesh filename=package://cer_rviz/../../../cer-gazebo/cer2/meshes/dae/sim_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 scale=0.001 0.001 0.001; visual mesh filename=package://cer_rviz/../../../cer-gazebo/cer2/meshes/dae/sim_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 scale=0.001 0.001 0.001
- added link r_wrist_slider_eq_link, mass 0.3; collision mesh filename=package://cer_rviz/../../../cer-gazebo/cer2/meshes/dae/sim_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 scale=0.001 0.001 0.001; visual mesh filename=package://cer_rviz/../../../cer-gazebo/cer2/meshes/dae/sim_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 scale=0.001 0.001 0.001
- added link torso_pin_eq_link, mass 1.5; collision mesh filename=package://cer_rviz/../../../cer-gazebo/cer2/meshes/dae/sim_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 scale=0.001 0.001 0.001; visual mesh filename=package://cer_rviz/../../../cer-gazebo/cer2/meshes/dae/sim_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 scale=0.001 0.001 0.001
- added link torso_platform_link, mass 1.5; collision mesh filename=package://cer_rviz/../../../cer-gazebo/cer2/meshes/dae/sim_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 scale=0.001 0.001 0.001; visual mesh filename=package://cer_rviz/../../../cer-gazebo/cer2/meshes/dae/sim_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 scale=0.001 0.001 0.001
- added link torso_slider_eq_link, mass 7.5; collision mesh filename=package://cer_rviz/../../../cer-gazebo/cer2/meshes/dae/sim_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 scale=0.001 0.001 0.001; visual mesh filename=package://cer_rviz/../../../cer-gazebo/cer2/meshes/dae/sim_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 scale=0.001 0.001 0.001
Joints:
- removed joint base_center_fixed_joint
- removed joint l_elbow
- removed joint l_hand_paddle_joint
- removed joint l_hand_thumb_joint
- removed joint l_shoulder_pitch
- removed joint l_shoulder_roll
- removed joint l_shoulder_yaw
- removed joint l_wrist_prosupination
- removed joint l_wrist_tripod_heave_eq
- removed joint l_wrist_tripod_pitch_eq
- removed joint l_wrist_tripod_roll_eq
- removed joint left_camera_fixed_joint
- removed joint lidar_fixed_joint
- removed joint mobile_base_l_wheel
- removed joint mobile_base_r_wheel
- removed joint neck_pitch
- removed joint neck_yaw
- removed joint oriented_xbk_yrg_zup_torso_tripod_platform_fixed_joint
- removed joint oriented_xfw_ylf_zup_torso_tripod_platform_fixed_joint
- removed joint r_elbow
- removed joint r_hand_paddle_joint
- removed joint r_hand_thumb_joint
- removed joint r_shoulder_pitch
- removed joint r_shoulder_roll
- removed joint r_shoulder_yaw
- removed joint r_wrist_prosupination
- removed joint r_wrist_tripod_heave_eq
- removed joint r_wrist_tripod_pitch_eq
- removed joint r_wrist_tripod_roll_eq
- removed joint right_camera_fixed_joint
- removed joint torso_tripod_heave_eq
- removed joint torso_tripod_pitch_eq
- removed joint torso_tripod_roll_eq
- removed joint torso_yaw
- added joint base_laser_fixed_joint: type fixed, parent mobile_base_body_link, child base_laser, origin xyz=0.07 0 0.031 rpy=0 0 0
- added joint l_elbow_joint: type revolute, parent l_upperarm_link, child l_elbow_sphere_link, origin xyz=0 0 0.1116 rpy=3.14159265359 0 1.57079632679, axis 0.0 -1.0 0.0, limit lower=0.0 upper=1.74532925199 effort=20.0 velocity=3.14
- added joint l_hand_paddle_distal_joint: type revolute, parent l_hand_paddle_proximal_link, child l_hand_paddle_distal_link, origin xyz=0 0.016328 -0.038746 rpy=0 0 0, axis -1.0 0.0 0.0, limit lower=0.0 upper=1.2217304764 effort=5.0 velocity=3.14
- added joint l_hand_paddle_proximal_joint: type revolute, parent l_hand_root_link, child l_hand_paddle_proximal_link, origin xyz=0 -0.012857 -0.112506 rpy=0 0 0, axis -1.0 0.0 0.0, limit lower=0.0 upper=1.2217304764 effort=5.0 velocity=3.14
- added joint l_hand_thumb_distal_joint: type revolute, parent l_hand_thumb_proximal_link, child l_hand_thumb_distal_link, origin xyz=0.001 -0.040525 -0.010986 rpy=0 0 0, axis 1.0 0.0 0.0, limit lower=0.0 upper=1.2217304764 effort=5.0 velocity=3.14
- added joint l_hand_thumb_proximal_joint: type revolute, parent l_hand_root_link, child l_hand_thumb_proximal_link, origin xyz=0 -0.039648 -0.075718 rpy=0 0 0, axis 1.0 0.0 0.0, limit lower=0.0 upper=1.0471975512 effort=5.0 velocity=3.14
- added joint l_shoulder_pitch_joint: type revolute, parent chest_link, child l_clavicle_link, origin xyz=-0.084 0.177 0.37 rpy=0 0 0, axis 0.0 -0.970296 -0.241922, limit lower=-0.523598775598 upper=1.57079632679 effort=30.0 velocity=3.14
- added joint l_shoulder_roll_joint: type revolute, parent l_clavicle_link, child l_shoulder_link, origin xyz=0 0 0 rpy=0 0 0, axis 1.0 0.0 0.0, limit lower=-0.174532925199 upper=1.308996939 effort=30.0 velocity=3.14
- added joint l_shoulder_yaw_joint: type revolute, parent l_shoulder_link, child l_upperarm_FT_sensor_link, origin xyz=0 0.034 -0.11 rpy=0 0 0, axis 0.0 0.0 1.0, limit lower=-1.57079632679 upper=1.57079632679 effort=15.0 velocity=3.14
- added joint l_upperarm_FT_sensor: type fixed, parent l_upperarm_FT_sensor_link, child l_upperarm_link, origin xyz=0 0 -0.0294 rpy=3.14159265359 0 1.57079632679
- added joint l_upperarm_FT_sensor_frame_fixed_joint: type fixed, parent l_upperarm_FT_sensor_link, child l_upperarm_FT_sensor_frame, origin xyz=0 0 -0.0294 rpy=3.14159265359 0 1.57079632679
- added joint l_wrist_heave_eq_joint: type prismatic, parent l_forearm_link, child l_wrist_slider_eq_link, origin xyz=0 0 0.071 rpy=0 0 0, axis 0.0 0.0 -1.0, limit lower=0.0 upper=0.13 effort=200.0 velocity=0.25
- added joint l_wrist_pitch_eq_joint: type revolute, parent l_wrist_cup_eq_link, child l_hand_root_link, origin xyz=0.045 0 0 rpy=0 0 0, axis 0.0 -1.0 0.0, limit lower=-0.523598775598 upper=0.523598775598 effort=10.0 velocity=3.14
- added joint l_wrist_pronosupination_joint: type revolute, parent l_elbow_sphere_link, child l_forearm_link, origin xyz=0 0 -0.071 rpy=0 0 0, axis 0.0 0.0 1.0, limit lower=-1.57079632679 upper=1.57079632679 effort=10.0 velocity=3.14
- added joint l_wrist_roll_eq_joint: type revolute, parent l_wrist_slider_eq_link, child l_wrist_cup_eq_link, origin xyz=-0.045 0 -0.291 rpy=0 0 0, axis 1.0 0.0 0.0, limit lower=-0.523598775598 upper=0.523598775598 effort=10.0 velocity=3.14
- added joint mobile_base_l_wheel_joint: type continuous, parent mobile_base_body_link, child mobile_base_l_tyre_link, origin xyz=0 0.139 0 rpy=0 0 0, axis 0.0 1.0 0.0, limit effort=100.0 velocity=30.0
- added joint mobile_base_r_wheel_joint: type continuous, parent mobile_base_body_link, child mobile_base_r_tyre_link, origin xyz=0 -0.139 0 rpy=0 0 0, axis 0.0 1.0 0.0, limit effort=100.0 velocity=30.0
- added joint multicamera_sensor_fixed_joint: type fixed, parent head_link, child multicamera_sensor, origin xyz=0.0515817 0 -0.06747 rpy=0 0 0
- added joint neck_pitch_joint: type revolute, parent chest_link, child neck_link, origin xyz=-0.094 0 0.4 rpy=0 0 0, axis 0.0 1.0 0.0, limit lower=-0.523598775598 upper=0.872664625997 effort=10.0 velocity=3.14
- added joint neck_yaw_joint: type revolute, parent neck_link, child head_link, origin xyz=0.0116795 0 0.15838 rpy=0 0 0, axis 0.173648 0.0 0.984808, limit lower=-1.3962634016 upper=1.3962634016 effort=10.0 velocity=3.14
- added joint oriented_xbk_yrg_zup_torso_platform_fixed_joint: type fixed, parent torso_platform_link, child oriented_xbk_yrg_zup_torso_platform, origin xyz=0 0 0 rpy=0 0 3.14159265359
- added joint oriented_xfw_ylf_zup_torso_platform_fixed_joint: type fixed, parent torso_platform_link, child oriented_xfw_ylf_zup_torso_platform, origin xyz=0 0 0 rpy=0 0 0
- added joint r_elbow_joint: type revolute, parent r_upperarm_link, child r_elbow_sphere_link, origin xyz=0 0 0.1116 rpy=3.14159265359 0 1.57079632679, axis 0.0 -1.0 0.0, limit lower=0.0 upper=1.74532925199 effort=20.0 velocity=3.14
- added joint r_hand_paddle_distal_joint: type revolute, parent r_hand_paddle_proximal_link, child r_hand_paddle_distal_link, origin xyz=0 -0.016328 -0.038746 rpy=0 0 0, axis 1.0 0.0 0.0, limit lower=0.0 upper=1.2217304764 effort=5.0 velocity=3.14
- added joint r_hand_paddle_proximal_joint: type revolute, parent r_hand_root_link, child r_hand_paddle_proximal_link, origin xyz=0 0.012857 -0.112506 rpy=0 0 0, axis 1.0 0.0 0.0, limit lower=0.0 upper=1.2217304764 effort=5.0 velocity=3.14
- added joint r_hand_thumb_distal_joint: type revolute, parent r_hand_thumb_proximal_link, child r_hand_thumb_distal_link, origin xyz=0 0.040525 -0.010986 rpy=0 0 0, axis -1.0 0.0 0.0, limit lower=0.0 upper=1.2217304764 effort=5.0 velocity=3.14
- added joint r_hand_thumb_proximal_joint: type revolute, parent r_hand_root_link, child r_hand_thumb_proximal_link, origin xyz=0 0.039648 -0.075718 rpy=0 0 0, axis -1.0 0.0 0.0, limit lower=0.0 upper=1.0471975512 effort=5.0 velocity=3.14
- added joint r_shoulder_pitch_joint: type revolute, parent chest_link, child r_clavicle_link, origin xyz=-0.084 -0.177 0.37 rpy=0 0 0, axis 0.0 -0.970296 0.241922, limit lower=-0.523598775598 upper=1.57079632679 effort=30.0 velocity=3.14
- added joint r_shoulder_roll_joint: type revolute, parent r_clavicle_link, child r_shoulder_link, origin xyz=0 0 0 rpy=0 0 0, axis -1.0 0.0 0.0, limit lower=-0.174532925199 upper=1.308996939 effort=30.0 velocity=3.14
- added joint r_shoulder_yaw_joint: type revolute, parent r_shoulder_link, child r_upperarm_FT_sensor_link, origin xyz=0 -0.034 -0.11 rpy=0 0 0, axis 0.0 0.0 -1.0, limit lower=-1.57079632679 upper=1.57079632679 effort=15.0 velocity=3.14
- added joint r_upperarm_FT_sensor: type fixed, parent r_upperarm_FT_sensor_link, child r_upperarm_link, origin xyz=0 0 -0.0294 rpy=3.14159265359 0 1.57079632679
- added joint r_upperarm_FT_sensor_frame_fixed_joint: type fixed, parent r_upperarm_FT_sensor_link, child r_upperarm_FT_sensor_frame, origin xyz=0 0 -0.0294 rpy=3.14159265359 0 1.57079632679
- added joint r_wrist_heave_eq_joint: type prismatic, parent r_forearm_link, child r_wrist_slider_eq_link, origin xyz=0 0 0.071 rpy=0 0 0, axis 0.0 0.0 -1.0, limit lower=0.0 upper=0.13 effort=200.0 velocity=0.25
- added joint r_wrist_pitch_eq_joint: type revolute, parent r_wrist_cup_eq_link, child r_hand_root_link, origin xyz=0 -0.045 0 rpy=0 0 -1.57079632679, axis 0.0 -1.0 0.0, limit lower=-0.523598775598 upper=0.523598775598 effort=10.0 velocity=3.14
- added joint r_wrist_pronosupination_joint: type revolute, parent r_elbow_sphere_link, child r_forearm_link, origin xyz=0 0 -0.071 rpy=0 0 0, axis 0.0 0.0 -1.0, limit lower=-1.57079632679 upper=1.57079632679 effort=10.0 velocity=3.14
- added joint r_wrist_roll_eq_joint: type revolute, parent r_wrist_slider_eq_link, child r_wrist_cup_eq_link, origin xyz=-0.045 0 -0.291 rpy=0 0 1.57079632679, axis 0.0 1.0 0.0, limit lower=-0.523598775598 upper=0.523598775598 effort=10.0 velocity=3.14
- added joint torso_heave_eq_joint: type prismatic, parent mobile_base_body_link, child torso_slider_eq_link, origin xyz=0.044 0 0.071 rpy=0 0 0, axis 0.0 0.0 1.0, limit lower=0.0 upper=0.17 effort=1200.0 velocity=0.5
- added joint torso_pitch_eq_joint: type revolute, parent torso_pin_eq_link, child torso_platform_link, origin xyz=0 0 0 rpy=3.14159265359 0 0, axis 0.0 1.0 0.0, limit lower=-0.523598775598 upper=0.523598775598 effort=50.0 velocity=3.14
- added joint torso_roll_eq_joint: type revolute, parent torso_slider_eq_link, child torso_pin_eq_link, origin xyz=0 0 0.399 rpy=3.14159265359 0 0, axis 1.0 0.0 0.0, limit lower=-0.523598775598 upper=0.523598775598 effort=50.0 velocity=3.14
- added joint torso_yaw_joint: type revolute, parent torso_platform_link, child chest_link, origin xyz=0 0 0 rpy=0 0 0, axis 0.0 0.0 1.0, limit lower=-1.0471975512 upper=1.0471975512 effort=30.0 velocity=3.14
- joint asus_xtion_fixed_joint: origin xyz=0.07702051 0 0.04662 rpy=0 0 0 -> xyz=0.0698802 0 0.04403 rpy=0 0 0; parent head -> head_link
- joint base_link_fixed_joint: origin xyz=0.074 0 0.63 rpy=0 0 0 -> xyz=0 0 0 rpy=0 0 0; parent mobile_base_body -> mobile_base_body_link
- joint gaze_fixed_joint: parent head -> head_link
- joint l_gripper_fixed_joint: origin xyz=0 -0.024941 -0.065778 rpy=3.141592653589793 1.221730955967807 -1.5707963267948968 -> xyz=0 -0.026917 -0.100456 rpy=3.14159265359 1.30899714732 -1.57079632679; parent l_hand_root -> l_hand_root_link
- joint l_hand_paddle_tip_fixed_joint: origin xyz=0 0 -0.084994 rpy=3.141592653589793 1.221730955967807 -1.5707963267948968 -> xyz=0 0.008959 -0.044226 rpy=3.14159265359 1.30899714732 -1.57079632679; parent l_hand_paddle -> l_hand_paddle_distal_link
- joint l_hand_thumb_tip_fixed_joint: origin xyz=0 -0.0513860000782 -0.0458929999125 rpy=3.141592653589793 1.2217309542643466 -1.570796326794897 -> xyz=-0.001 -0.028617 -0.014073 rpy=3.14159265359 1.30899714732 -1.57079632679; parent l_hand_thumb -> l_hand_thumb_distal_link
- joint l_wrist_fixed_joint: origin xyz=0 -0.001 0 rpy=0 0 0 -> xyz=0 0 0 rpy=3.14159265359 0 -1.57079632679; parent l_hand_root -> l_hand_root_link
- joint oriented_l_wrist_tripodbase_fixed_joint: origin xyz=0 0 0 rpy=3.141592653589793 0 -1.5707963267948966 -> xyz=0 0 -0.22 rpy=3.14159265359 0 -1.57079632679; parent l_wrist_tripod_base -> l_forearm_link
- joint oriented_r_wrist_tripodbase_fixed_joint: origin xyz=0 0 0 rpy=3.141592653589793 0 1.5707963267948966 -> xyz=0 0 -0.22 rpy=3.14159265359 0 1.57079632679; parent r_wrist_tripod_base -> r_forearm_link
- joint r_gripper_fixed_joint: origin xyz=0 0.022941 -0.065778 rpy=0 1.221730955967806 1.5707963267948957 -> xyz=0 0.026917 -0.100456 rpy=0 1.30899714732 1.57079632679; parent r_hand_root -> r_hand_root_link
- joint r_hand_paddle_tip_fixed_joint: origin xyz=0 0 -0.084994 rpy=0 1.221730955967806 1.5707963267948957 -> xyz=0 -0.008959 -0.044226 rpy=0 1.30899714732 1.57079632679; parent r_hand_paddle -> r_hand_paddle_distal_link
- joint r_hand_thumb_tip_fixed_joint: origin xyz=0 0.051386 -0.045893 rpy=0 1.221730955967806 1.5707963267948957 -> xyz=0 0.028617 -0.014073 rpy=0 1.30899714732 1.57079632679; parent r_hand_thumb -> r_hand_thumb_distal_link
- joint r_wrist_fixed_joint: origin xyz=0 -0.001 0 rpy=0 0 0 -> xyz=0 0 0 rpy=3.14159265359 0 1.57079632679; parent r_hand_root -> r_hand_root_link
- joint torso_fixed_joint: origin xyz=-0.042 0 0.17 rpy=0 0 0 -> xyz=-0.042 0 0.185 rpy=0 0 0; parent torso_chest -> chest_link
