Commit message: added z translation for cer odometry, fixed reference frame names

File: app/robots/CER01/cer.urdf (robot description, URDF)
Before this commit: robot SIM_CER_ROBOT, 55 links, 54 joints
Joints:
- joint base_laser_fixed_joint: origin xyz=0.07 0 0.031 rpy=0 0 0 -> xyz=0.07 0 0.031 rpy=0 0 -1.57

Commit message: added some frames to urdf

File: app/robots/CER01/cer.urdf (robot description, URDF)
Before this commit: robot SIM_CER_ROBOT, 55 links, 54 joints
Links:
- added link base_laser_rp
- added link camera_link
- added link mobile_base_body
Joints:
- added joint custom1_joint: type fixed, parent asus_xtion, child camera_link, origin xyz=0.0 0 0.0 rpy=0 0 0
- added joint custom2_joint: type fixed, parent mobile_base_body_link, child mobile_base_body, origin xyz=0.0 0 0.0 rpy=0 0 0
- added joint custom3_joint: type fixed, parent base_laser, child base_laser_rp, origin xyz=0.0 0 0.0 rpy=0 0 -1.57

Commit message: urdf update

File: app/robots/CER01/cer.urdf (robot description, URDF)
Before this commit: robot SIM_CER_ROBOT, 58 links, 57 joints
Links:
- removed link asus_xtion
- removed link base_laser
- removed link base_laser_rp
- removed link camera_link
- removed link mobile_base_body
- removed link multicamera_sensor
- removed link oriented_l_wrist_tripodbase
- removed link oriented_r_wrist_tripodbase
- removed link oriented_xbk_yrg_zup_torso_platform
- removed link oriented_xfw_ylf_zup_torso_platform
- added link depth
- added link depth_center
- added link depth_rgb
- added link head_leopard_cyclopic
- added link head_leopard_left
- added link head_leopard_right
- added link l_wrist_tripod_root
- added link mobile_base_lidar
- added link r_wrist_tripod_root
- added link torso_tripod_root
- link chest_link: geometry collision mesh filename=package://cer/meshes/dae/sim_cer_chest.dae scale=0.001 0.001 0.001; visual mesh filename=package://cer/meshes/dae/sim_cer_chest.dae scale=0.001 0.001 0.001
- link head_link: geometry collision mesh filename=package://cer/meshes/dae/sim_cer_head.dae scale=0.001 0.001 0.001; visual mesh filename=package://cer/meshes/dae/sim_cer_head.dae scale=0.001 0.001 0.001
- link l_clavicle_link: geometry collision mesh filename=package://cer/meshes/dae/sim_cer_l_clavicle.dae scale=0.001 0.001 0.001; visual mesh filename=package://cer/meshes/dae/sim_cer_l_clavicle.dae scale=0.001 0.001 0.001
- link l_elbow_sphere_link: geometry collision mesh filename=package://cer/meshes/dae/sim_cer_l_elbow_sphere.dae scale=0.001 0.001 0.001; visual mesh filename=package://cer/meshes/dae/sim_cer_l_elbow_sphere.dae scale=0.001 0.001 0.001
- link l_forearm_link: geometry collision mesh filename=package://cer/meshes/dae/sim_cer_l_forearm.dae scale=0.001 0.001 0.001; visual mesh filename=package://cer/meshes/dae/sim_cer_l_forearm.dae scale=0.001 0.001 0.001
- link l_hand_paddle_distal_link: geometry collision mesh filename=package://cer/meshes/dae/sim_cer_l_hand_paddle_distal.dae scale=0.001 0.001 0.001; visual mesh filename=package://cer/meshes/dae/sim_cer_l_hand_paddle_distal.dae scale=0.001 0.001 0.001
- link l_hand_paddle_proximal_link: geometry collision mesh filename=package://cer/meshes/dae/sim_cer_l_hand_paddle_proximal.dae scale=0.001 0.001 0.001; visual mesh filename=package://cer/meshes/dae/sim_cer_l_hand_paddle_proximal.dae scale=0.001 0.001 0.001
- link l_hand_root_link: geometry collision mesh filename=package://cer/meshes/dae/sim_cer_l_hand_root.dae scale=0.001 0.001 0.001; visual mesh filename=package://cer/meshes/dae/sim_cer_l_hand_root.dae scale=0.001 0.001 0.001
- link l_hand_thumb_distal_link: geometry collision mesh filename=package://cer/meshes/dae/sim_cer_l_hand_thumb_distal.dae scale=0.001 0.001 0.001; visual mesh filename=package://cer/meshes/dae/sim_cer_l_hand_thumb_distal.dae scale=0.001 0.001 0.001
- link l_hand_thumb_proximal_link: geometry collision mesh filename=package://cer/meshes/dae/sim_cer_l_hand_thumb_proximal.dae scale=0.001 0.001 0.001; visual mesh filename=package://cer/meshes/dae/sim_cer_l_hand_thumb_proximal.dae scale=0.001 0.001 0.001
- link l_shoulder_link: geometry collision mesh filename=package://cer/meshes/dae/sim_cer_l_shoulder.dae scale=0.001 0.001 0.001; visual mesh filename=package://cer/meshes/dae/sim_cer_l_shoulder.dae scale=0.001 0.001 0.001
- link l_upperarm_FT_sensor_link: geometry collision mesh filename=package://cer/meshes/dae/sim_cer_l_upperarm_sensor.dae scale=0.001 0.001 0.001; visual mesh filename=package://cer/meshes/dae/sim_cer_l_upperarm_sensor.dae scale=0.001 0.001 0.001
- link l_upperarm_link: geometry collision mesh filename=package://cer/meshes/dae/sim_cer_l_upperarm.dae scale=0.001 0.001 0.001; visual mesh filename=package://cer/meshes/dae/sim_cer_l_upperarm.dae scale=0.001 0.001 0.001
- link l_wrist_cup_eq_link: geometry collision mesh filename=package://cer/meshes/dae/sim_cer_l_wrist_cup_eq.dae scale=0.001 0.001 0.001; visual mesh filename=package://cer/meshes/dae/sim_cer_l_wrist_cup_eq.dae scale=0.001 0.001 0.001
- link l_wrist_slider_eq_link: geometry collision mesh filename=package://cer/meshes/dae/sim_cer_l_wrist_slider.dae scale=0.001 0.001 0.001; visual mesh filename=package://cer/meshes/dae/sim_cer_l_wrist_slider.dae scale=0.001 0.001 0.001
- link mobile_base_body_link: geometry collision mesh filename=package://cer/meshes/dae/sim_cer_mobilebase_body.dae scale=0.001 0.001 0.001; visual mesh filename=package://cer/meshes/dae/sim_cer_mobilebase_body.dae scale=0.001 0.001 0.001
- link mobile_base_l_tyre_link: geometry collision cylinder length=0.005 radius=0.16; visual mesh filename=package://cer/meshes/dae/sim_cer_mobilebase_l_tyre.dae scale=0.001 0.001 0.001
- link mobile_base_r_tyre_link: geometry collision cylinder length=0.005 radius=0.16; visual mesh filename=package://cer/meshes/dae/sim_cer_mobilebase_r_tyre.dae scale=0.001 0.001 0.001
- link neck_link: geometry collision mesh filename=package://cer/meshes/dae/sim_cer_neck.dae scale=0.001 0.001 0.001; visual mesh filename=package://cer/meshes/dae/sim_cer_neck.dae scale=0.001 0.001 0.001
- link r_clavicle_link: geometry collision mesh filename=package://cer/meshes/dae/sim_cer_r_clavicle.dae scale=0.001 0.001 0.001; visual mesh filename=package://cer/meshes/dae/sim_cer_r_clavicle.dae scale=0.001 0.001 0.001
- link r_elbow_sphere_link: geometry collision mesh filename=package://cer/meshes/dae/sim_cer_r_elbow_sphere.dae scale=0.001 0.001 0.001; visual mesh filename=package://cer/meshes/dae/sim_cer_r_elbow_sphere.dae scale=0.001 0.001 0.001
- link r_forearm_link: geometry collision mesh filename=package://cer/meshes/dae/sim_cer_r_forearm.dae scale=0.001 0.001 0.001; visual mesh filename=package://cer/meshes/dae/sim_cer_r_forearm.dae scale=0.001 0.001 0.001
- link r_hand_paddle_distal_link: geometry collision mesh filename=package://cer/meshes/dae/sim_cer_r_hand_paddle_distal.dae scale=0.001 0.001 0.001; visual mesh filename=package://cer/meshes/dae/sim_cer_r_hand_paddle_distal.dae scale=0.001 0.001 0.001
- link r_hand_paddle_proximal_link: geometry collision mesh filename=package://cer/meshes/dae/sim_cer_r_hand_paddle_proximal.dae scale=0.001 0.001 0.001; visual mesh filename=package://cer/meshes/dae/sim_cer_r_hand_paddle_proximal.dae scale=0.001 0.001 0.001
- link r_hand_root_link: geometry collision mesh filename=package://cer/meshes/dae/sim_cer_r_hand_root.dae scale=0.001 0.001 0.001; visual mesh filename=package://cer/meshes/dae/sim_cer_r_hand_root.dae scale=0.001 0.001 0.001
- link r_hand_thumb_distal_link: geometry collision mesh filename=package://cer/meshes/dae/sim_cer_r_hand_thumb_distal.dae scale=0.001 0.001 0.001; visual mesh filename=package://cer/meshes/dae/sim_cer_r_hand_thumb_distal.dae scale=0.001 0.001 0.001
- link r_hand_thumb_proximal_link: geometry collision mesh filename=package://cer/meshes/dae/sim_cer_r_hand_thumb_proximal.dae scale=0.001 0.001 0.001; visual mesh filename=package://cer/meshes/dae/sim_cer_r_hand_thumb_proximal.dae scale=0.001 0.001 0.001
- link r_shoulder_link: geometry collision mesh filename=package://cer/meshes/dae/sim_cer_r_shoulder.dae scale=0.001 0.001 0.001; visual mesh filename=package://cer/meshes/dae/sim_cer_r_shoulder.dae scale=0.001 0.001 0.001
- link r_upperarm_FT_sensor_link: geometry collision mesh filename=package://cer/meshes/dae/sim_cer_r_upperarm_sensor.dae scale=0.001 0.001 0.001; visual mesh filename=package://cer/meshes/dae/sim_cer_r_upperarm_sensor.dae scale=0.001 0.001 0.001
- link r_upperarm_link: geometry collision mesh filename=package://cer/meshes/dae/sim_cer_r_upperarm.dae scale=0.001 0.001 0.001; visual mesh filename=package://cer/meshes/dae/sim_cer_r_upperarm.dae scale=0.001 0.001 0.001
- link r_wrist_cup_eq_link: geometry collision mesh filename=package://cer/meshes/dae/sim_cer_r_wrist_cup_eq.dae scale=0.001 0.001 0.001; visual mesh filename=package://cer/meshes/dae/sim_cer_r_wrist_cup_eq.dae scale=0.001 0.001 0.001
- link r_wrist_slider_eq_link: geometry collision mesh filename=package://cer/meshes/dae/sim_cer_r_wrist_slider.dae scale=0.001 0.001 0.001; visual mesh filename=package://cer/meshes/dae/sim_cer_r_wrist_slider.dae scale=0.001 0.001 0.001
- link torso_pin_eq_link: geometry collision mesh filename=package://cer/meshes/dae/sim_cer_torso_pin_eq.dae scale=0.001 0.001 0.001; visual mesh filename=package://cer/meshes/dae/sim_cer_torso_pin_eq.dae scale=0.001 0.001 0.001
- link torso_platform_link: geometry collision mesh filename=package://cer/meshes/dae/sim_cer_torso_platform.dae scale=0.001 0.001 0.001; visual mesh filename=package://cer/meshes/dae/sim_cer_torso_platform.dae scale=0.001 0.001 0.001
- link torso_slider_eq_link: geometry collision mesh filename=package://cer/meshes/dae/sim_cer_torso_slider_eq.dae scale=0.001 0.001 0.001; visual mesh filename=package://cer/meshes/dae/sim_cer_torso_slider_eq.dae scale=0.001 0.001 0.001
Joints:
- removed joint asus_xtion_fixed_joint
- removed joint base_laser_fixed_joint
- removed joint custom1_joint
- removed joint custom2_joint
- removed joint custom3_joint
- removed joint multicamera_sensor_fixed_joint
- removed joint oriented_l_wrist_tripodbase_fixed_joint
- removed joint oriented_r_wrist_tripodbase_fixed_joint
- removed joint oriented_xbk_yrg_zup_torso_platform_fixed_joint
- removed joint oriented_xfw_ylf_zup_torso_platform_fixed_joint
- added joint depth_center_fixed_joint: type fixed, parent head_link, child depth_center, origin xyz=0.0598756 0 0.04402 rpy=-1.57079632679 0 -1.57079632679
- added joint depth_fixed_joint: type fixed, parent head_link, child depth, origin xyz=0.0598814 0.0444871 0.04402 rpy=-1.57079632679 0 -1.57079632679
- added joint depth_rgb_fixed_joint: type fixed, parent head_link, child depth_rgb, origin xyz=0.0598814 0.0184871 0.04402 rpy=-1.57079632679 0 -1.57079632679
- added joint head_leopard_cyclopic_fixed_joint: type fixed, parent head_link, child head_leopard_cyclopic, origin xyz=0.0521666 0 -0.06748 rpy=-1.57079632679 0 -1.57079632679
- added joint head_leopard_left_fixed_joint: type fixed, parent head_link, child head_leopard_left, origin xyz=0.0521666 0.0335105 -0.06748 rpy=-1.57079632679 0 -1.57079632679
- added joint head_leopard_right_fixed_joint: type fixed, parent head_link, child head_leopard_right, origin xyz=0.0521666 -0.0335105 -0.06748 rpy=-1.57079632679 0 -1.57079632679
- added joint l_wrist_tripod_root_fixed_joint: type fixed, parent l_forearm_link, child l_wrist_tripod_root, origin xyz=0 0 -0.22 rpy=3.14159265359 0 -1.57079632679
- added joint mobile_base_lidar_fixed_joint: type fixed, parent mobile_base_body_link, child mobile_base_lidar, origin xyz=0.07 0 0.031 rpy=0 0 0
- added joint r_wrist_tripod_root_fixed_joint: type fixed, parent r_forearm_link, child r_wrist_tripod_root, origin xyz=0 0 -0.22 rpy=3.14159265359 0 1.57079632679
- added joint torso_tripod_root_fixed_joint: type fixed, parent torso_platform_link, child torso_tripod_root, origin xyz=0 0 0 rpy=0 0 3.14159265359
- joint gaze_fixed_joint: origin xyz=0 0 0 rpy=0 0 0 -> xyz=0.0494817 0 -0.01388 rpy=-1.57079632679 0 -1.57079632679
- joint l_hand_thumb_distal_joint: origin xyz=0.001 -0.040525 -0.010986 rpy=0 0 0 -> xyz=0.000255 -0.040525 -0.010986 rpy=0 0 0
- joint l_hand_thumb_tip_fixed_joint: origin xyz=-0.001 -0.028617 -0.014073 rpy=3.14159265359 1.30899714732 -1.57079632679 -> xyz=-0.000255 -0.028617 -0.014073 rpy=3.14159265359 1.30899714732 -1.57079632679
- joint l_wrist_pitch_eq_joint: origin xyz=0.045 0 0 rpy=0 0 0 -> xyz=0.032 0 0 rpy=0 0 0
- joint l_wrist_roll_eq_joint: origin xyz=-0.045 0 -0.291 rpy=0 0 0 -> xyz=-0.032 0 -0.291 rpy=0 0 0
- joint r_wrist_pitch_eq_joint: origin xyz=0 -0.045 0 rpy=0 0 -1.57079632679 -> xyz=0 -0.032 0 rpy=0 0 -1.57079632679
- joint r_wrist_roll_eq_joint: origin xyz=-0.045 0 -0.291 rpy=0 0 1.57079632679 -> xyz=-0.032 0 -0.291 rpy=0 0 1.57079632679
