Commit message: Fix double laser in cer.urdf of CER03

File: app/robots/CER03/cer.urdf (robot description, URDF)
Before this commit: robot SIM_CER_ROBOT, 58 links, 57 joints
Links:
- removed link mobile_base_lidar
- added link mobile_base_double_lidar
- added link mobile_base_lidar_B
- added link mobile_base_lidar_F
Joints:
- removed joint mobile_base_lidar_fixed_joint
- added joint mobile_base_double_lidar_fixed_joint: type fixed, parent mobile_base_body_link, child mobile_base_double_lidar, origin xyz=0.0 0 0.031 rpy=0 0 0
- added joint mobile_base_lidar_B_fixed_joint: type fixed, parent mobile_base_body_link, child mobile_base_lidar_B, origin xyz=-0.085 0 0.031 rpy=0 0 3.14
- added joint mobile_base_lidar_F_fixed_joint: type fixed, parent mobile_base_body_link, child mobile_base_lidar_F, origin xyz=0.07 0 0.031 rpy=0 0 0
